File: vga_ambilight_throughhole.sch (EAGLE design)
At the start: 14 parts, among them IC1 QUAD_OPAMPD

Commit message: commit
Parts:
- added C1: 10uf, adafruit:C-USC1206
- added C2: 0.1uf, adafruit:C-USC1206
Connections:
- net GND: now also C1.2, C2.2
- net VCC: now also C1.1, C2.1
Changed lines of the file:
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@@
 <part name="JP3" library="sparkfun" deviceset="M04" device="PTH"/>
 <part name="JP4" library="sparkfun" deviceset="M04" device="PTH"/>
-<part name="GND3" library="sparkfun" deviceset="GND" device=""/>
 <part name="P+3" library="supply1" deviceset="+12V" device=""/>
 <part name="J1" library="con-jack" deviceset="DCJ0303" device=""/>
 <part name="P+4" library="supply1" deviceset="+12V" device=""/>
+<part name="GND3" library="sparkfun" deviceset="GND" device=""/>
 <part name="GND4" library="sparkfun" deviceset="GND" device=""/>
+<part name="C1" library="adafruit" deviceset="C-US" device="C1206" value="10uf"/>
+<part name="C2" library="adafruit" deviceset="C-US" device="C1206" value="0.1uf"/>
+<part name="P+5" library="sparkfun" deviceset="VCC" device=""/>
+<part name="GND5" library="sparkfun" deviceset="GND" device=""/>
 </parts>
 <sheets>
@@
 <instance part="JP3" gate="G$1" x="81.28" y="-7.62" rot="R180"/>
 <instance part="JP4" gate="G$1" x="73.66" y="-7.62" rot="R180"/>
-<instance part="GND3" gate="1" x="114.3" y="27.94"/>
 <instance part="P+3" gate="1" x="66.04" y="2.54"/>
 <instance part="J1" gate="G$1" x="30.48" y="0"/>
 <instance part="P+4" gate="1" x="40.64" y="7.62"/>
-<instance part="GND4" gate="1" x="40.64" y="-10.16"/>
+<instance part="GND3" gate="1" x="40.64" y="-10.16"/>
+<instance part="GND4" gate="1" x="114.3" y="27.94"/>
+<instance part="C1" gate="G$1" x="114.3" y="7.62"/>
+<instance part="C2" gate="G$1" x="121.92" y="7.62"/>
+<instance part="P+5" gate="1" x="114.3" y="15.24"/>
+<instance part="GND5" gate="1" x="114.3" y="-5.08"/>
 </instances>
 <busses>
@@
 </segment>
 <segment>
+<pinref part="J1" gate="G$1" pin="2"/>
+<wire x1="38.1" y1="0" x2="40.64" y2="0" width="0.1524" layer="91"/>
+<wire x1="40.64" y1="0" x2="40.64" y2="-2.54" width="0.1524" layer="91"/>
+<pinref part="J1" gate="G$1" pin="3"/>
+<wire x1="40.64" y1="-2.54" x2="40.64" y2="-7.62" width="0.1524" layer="91"/>
+<wire x1="38.1" y1="-2.54" x2="40.64" y2="-2.54" width="0.1524" layer="91"/>
+<pinref part="GND3" gate="1" pin="GND"/>
+</segment>
+<segment>
 <pinref part="Q3" gate="G$1" pin="S"/>
 <wire x1="114.3" y1="35.56" x2="114.3" y2="33.02" width="0.1524" layer="91"/>
@@
 <junction x="119.38" y="53.34"/>
 <wire x1="114.3" y1="33.02" x2="119.38" y2="33.02" width="0.1524" layer="91"/>
-<pinref part="GND3" gate="1" pin="GND"/>
+<pinref part="GND4" gate="1" pin="GND"/>
 </segment>
 <segment>
-<pinref part="J1" gate="G$1" pin="2"/>
-<wire x1="38.1" y1="0" x2="40.64" y2="0" width="0.1524" layer="91"/>
-<wire x1="40.64" y1="0" x2="40.64" y2="-2.54" width="0.1524" layer="91"/>
-<pinref part="J1" gate="G$1" pin="3"/>
-<wire x1="40.64" y1="-2.54" x2="40.64" y2="-7.62" width="0.1524" layer="91"/>
-<wire x1="38.1" y1="-2.54" x2="40.64" y2="-2.54" width="0.1524" layer="91"/>
-<pinref part="GND4" gate="1" pin="GND"/>
+<pinref part="C2" gate="G$1" pin="2"/>
+<wire x1="121.92" y1="2.54" x2="121.92" y2="0" width="0.1524" layer="91"/>
+<wire x1="121.92" y1="0" x2="114.3" y2="0" width="0.1524" layer="91"/>
+<pinref part="C1" gate="G$1" pin="2"/>
+<wire x1="114.3" y1="0" x2="114.3" y2="2.54" width="0.1524" layer="91"/>
+<pinref part="GND5" gate="1" pin="GND"/>
+<wire x1="114.3" y1="2.54" x2="114.3" y2="0" width="0.1524" layer="91"/>
+<junction x="114.3" y="0"/>
+<wire x1="114.3" y1="0" x2="114.3" y2="-2.54" width="0.1524" layer="91"/>
 </segment>
 </net>
@@
 <pinref part="P+1" gate="1" pin="VCC"/>
 </segment>
+<segment>
+<pinref part="C1" gate="G$1" pin="1"/>
+<pinref part="P+5" gate="1" pin="VCC"/>
+<wire x1="114.3" y1="10.16" x2="114.3" y2="12.7" width="0.1524" layer="91"/>
+<wire x1="114.3" y1="15.24" x2="114.3" y2="12.7" width="0.1524" layer="91"/>
+<pinref part="C2" gate="G$1" pin="1"/>
+<wire x1="114.3" y1="12.7" x2="121.92" y2="12.7" width="0.1524" layer="91"/>
+<wire x1="121.92" y1="12.7" x2="121.92" y2="10.16" width="0.1524" layer="91"/>
+<junction x="114.3" y="12.7"/>
+</segment>
 </net>
