File: vga_ambilight_throughhole.brd (EAGLE design)
At the start: 46.4 x 40.6 mm, 16 parts, among them IC1 QUAD_OPAMPD

Commit message: commit
Parts:
- R1, R2, R3: device adafruit:M1206 -> adafruit:M0805
Other:
- board text added: "Analog ambient light adapter"
- board text added: "Jeremy Ruhland"
Changed lines of the file:
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@@
 <setting verticaltext="up"/>
 </settings>
-<grid distance="0.05" unitdist="inch" unit="inch" style="lines" multiple="1" display="no" altdistance="0.025" altunitdist="inch" altunit="inch"/>
+<grid distance="0.05" unitdist="inch" unit="inch" style="lines" multiple="1" display="no" altdistance="0.0125" altunitdist="inch" altunit="inch"/>
 <layers>
 <layer number="1" name="Top" color="4" fill="1" visible="yes" active="yes"/>
@@
 <text x="26.67" y="50.8" size="0.6096" layer="121">G</text>
 <text x="29.21" y="50.8" size="0.6096" layer="121">B</text>
+<text x="10.16" y="77.47" size="0.8128" layer="121">Analog ambient light adapter</text>
+<text x="10.16" y="76.2" size="0.6096" layer="121">Jeremy Ruhland</text>
 </plain>
 <attributes>
@@
 <attribute name="VALUE" x="31.75" y="56.515" size="1.27" layer="27" rot="R180"/>
 </element>
-<element name="R1" library="adafruit" package="M1206" value="" x="22.225" y="58.42" smashed="yes" rot="R270">
+<element name="R1" library="adafruit" package="M0805" value="" x="22.225" y="58.42" smashed="yes" rot="R270">
 <attribute name="NAME" x="23.495" y="59.69" size="1.27" layer="25" rot="R270"/>
 <attribute name="VALUE" x="19.685" y="59.69" size="1.27" layer="27" rot="R270"/>
 </element>
-<element name="R2" library="adafruit" package="M1206" value="" x="26.035" y="58.42" smashed="yes" rot="R270">
+<element name="R2" library="adafruit" package="M0805" value="" x="26.035" y="58.42" smashed="yes" rot="R270">
 <attribute name="NAME" x="27.305" y="59.69" size="1.27" layer="25" rot="R270"/>
 <attribute name="VALUE" x="23.495" y="59.69" size="1.27" layer="27" rot="R270"/>
 </element>
-<element name="R3" library="adafruit" package="M1206" value="" x="29.845" y="58.42" smashed="yes" rot="R270">
+<element name="R3" library="adafruit" package="M0805" value="" x="29.845" y="58.42" smashed="yes" rot="R270">
 <attribute name="NAME" x="31.115" y="59.69" size="1.27" layer="25" rot="R270"/>
 <attribute name="VALUE" x="27.305" y="59.69" size="1.27" layer="27" rot="R270"/>
@@
 <wire x1="23.368" y1="66.04" x2="29.464" y2="59.944" width="0.4064" layer="1"/>
 <wire x1="23.368" y1="67.564" x2="23.368" y2="66.04" width="0.4064" layer="1"/>
-<wire x1="29.464" y1="59.944" x2="29.845" y2="59.82" width="0.4064" layer="1"/>
+<wire x1="29.464" y1="59.944" x2="29.845" y2="59.37" width="0.4064" layer="1"/>
 <wire x1="23.368" y1="68.072" x2="22.352" y2="68.072" width="0.4064" layer="1"/>
 <wire x1="22.352" y1="68.072" x2="22.225" y2="68.005" width="0.4064" layer="1"/>
@@
 <wire x1="23.368" y1="62.992" x2="23.495" y2="62.805" width="0.4064" layer="1"/>
 <wire x1="23.495" y1="62.805" x2="26.035" y2="60.265" width="0.4064" layer="1"/>
-<wire x1="26.035" y1="60.265" x2="26.035" y2="59.82" width="0.4064" layer="1"/>
+<wire x1="26.035" y1="60.265" x2="26.035" y2="59.37" width="0.4064" layer="1"/>
 </signal>
 <signal name="N$8">
@@
 <contactref element="IC1" pad="1"/>
 <contactref element="R1" pad="1"/>
-<wire x1="21.844" y1="59.944" x2="22.225" y2="59.82" width="0.4064" layer="1"/>
 <wire x1="15.875" y1="62.805" x2="15.875" y2="61.595" width="0.4064" layer="1"/>
 <wire x1="15.875" y1="62.805" x2="17.145" y2="62.805" width="0.4064" layer="1"/>
@@
 <wire x1="18.415" y1="60.96" x2="19.555" y2="59.82" width="0.4064" layer="1"/>
 <wire x1="19.555" y1="59.82" x2="22.225" y2="59.82" width="0.4064" layer="1"/>
+<wire x1="22.225" y1="59.82" x2="22.225" y2="59.37" width="0.4064" layer="1"/>
 </signal>
 <signal name="R">
@@
 <contactref element="X1" pad="15"/>
 <contactref element="X2" pad="15"/>
-<wire x1="7.62" y1="68.072" x2="4.064" y2="68.072" width="0.4064" layer="16"/>
-<wire x1="17.78" y1="57.912" x2="7.62" y2="68.072" width="0.4064" layer="16"/>
-<wire x1="20.32" y1="57.912" x2="17.78" y2="57.912" width="0.4064" layer="16"/>
-<wire x1="20.828" y1="58.42" x2="20.32" y2="57.912" width="0.4064" layer="16"/>
-<wire x1="30.988" y1="58.42" x2="20.828" y2="58.42" width="0.4064" layer="1"/>
-<wire x1="33.528" y1="55.88" x2="30.988" y2="58.42" width="0.4064" layer="1"/>
-<wire x1="33.528" y1="51.816" x2="33.528" y2="55.88" width="0.4064" layer="1"/>
-<wire x1="34.544" y1="50.8" x2="33.528" y2="51.816" width="0.4064" layer="1"/>
-<wire x1="37.084" y1="50.8" x2="34.544" y2="50.8" width="0.4064" layer="1"/>
-<wire x1="4.064" y1="68.072" x2="3.81" y2="67.9196" width="0.4064" layer="16"/>
-<wire x1="37.084" y1="50.8" x2="37.465" y2="50.8254" width="0.4064" layer="1"/>
-<via x="20.828" y="58.42" extent="1-16" drill="0.3048"/>
+<wire x1="3.81" y1="67.9196" x2="7.0104" y2="67.9196" width="0.4064" layer="16"/>
+<wire x1="7.0104" y1="67.9196" x2="11.43" y2="63.5" width="0.4064" layer="16"/>
+<wire x1="11.43" y1="63.5" x2="11.43" y2="61.9125" width="0.4064" layer="16"/>
+<wire x1="11.43" y1="61.9125" x2="17.145" y2="56.1975" width="0.4064" layer="16"/>
+<wire x1="17.145" y1="56.1975" x2="31.4325" y2="56.1975" width="0.4064" layer="16"/>
+<wire x1="37.465" y1="50.8254" x2="33.9471" y2="50.8254" width="0.4064" layer="1"/>
+<wire x1="33.9471" y1="50.8254" x2="32.385" y2="52.3875" width="0.4064" layer="1"/>
+<wire x1="32.385" y1="52.3875" x2="32.385" y2="55.245" width="0.4064" layer="1"/>
+<wire x1="32.385" y1="55.245" x2="31.4325" y2="56.1975" width="0.4064" layer="1"/>
+<via x="31.4325" y="56.1975" extent="1-16" drill="0.3048"/>
 </signal>
 <signal name="N$10">
@@
 <wire x1="34.925" y1="71.755" x2="31.115" y2="71.755" width="0.4064" layer="16"/>
 <wire x1="31.115" y1="71.755" x2="30.48" y2="72.39" width="0.4064" layer="16"/>
-<via x="30.48" y="72.39" extent="1-16" drill="0.5"/>
+<via x="30.48" y="72.39" extent="1-16" drill="0.3048"/>
 <wire x1="5.715" y1="71.755" x2="29.845" y2="71.755" width="0.4064" layer="1"/>
 <wire x1="29.845" y1="71.755" x2="30.48" y2="72.39" width="0.4064" layer="1"/>
@@
 <wire x1="4.445" y1="73.025" x2="22.225" y2="73.025" width="0.4064" layer="1"/>
 <wire x1="22.225" y1="73.025" x2="22.86" y2="73.66" width="0.4064" layer="1"/>
-<via x="22.86" y="73.66" extent="1-16" drill="0.5"/>
+<via x="22.86" y="73.66" extent="1-16" drill="0.3048"/>
 <wire x1="22.86" y1="73.66" x2="22.86" y2="73.152" width="0.4064" layer="16"/>
 <wire x1="22.86" y1="73.152" x2="32.512" y2="63.5" width="0.4064" layer="16"/>
@@
 <wire x1="22.352" y1="56.896" x2="22.86" y2="56.388" width="0.4064" layer="1"/>
 <wire x1="22.86" y1="54.864" x2="23.175" y2="54.44" width="0.4064" layer="1"/>
-<wire x1="22.352" y1="56.896" x2="22.225" y2="57.02" width="0.4064" layer="1"/>
+<wire x1="22.352" y1="56.896" x2="22.225" y2="57.47" width="0.4064" layer="1"/>
 </signal>
 <signal name="N$13">
@@
 <wire x1="26.416" y1="56.896" x2="26.924" y2="56.388" width="0.4064" layer="1"/>
 <wire x1="26.924" y1="54.864" x2="26.985" y2="54.44" width="0.4064" layer="1"/>
-<wire x1="26.416" y1="56.896" x2="26.035" y2="57.02" width="0.4064" layer="1"/>
+<wire x1="26.416" y1="56.896" x2="26.035" y2="57.47" width="0.4064" layer="1"/>
 </signal>
 <signal name="N$16">
@@
 <wire x1="29.972" y1="56.896" x2="30.48" y2="56.388" width="0.4064" layer="1"/>
 <wire x1="30.48" y1="54.864" x2="30.795" y2="54.44" width="0.4064" layer="1"/>
-<wire x1="29.972" y1="56.896" x2="29.845" y2="57.02" width="0.4064" layer="1"/>
+<wire x1="29.972" y1="56.896" x2="29.845" y2="57.47" width="0.4064" layer="1"/>
 </signal>
 <signal name="R_PWR">

Commit message: commit
Routing:
- net N$15: track 64.9 -> 66.3 mm
- net GND: vias 1 -> 5
- removed copper zone on layer 16, net N$17
- removed copper zone on layer 1, net N$18
Changed lines of the file:
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@@
 <contactref element="X1" pad="10"/>
 <contactref element="X2" pad="10"/>
-<polygon width="0.8128" layer="16">
+<polygon width="0.8128" layer="16" isolate="0.3048">
 <vertex x="43.18" y="40.005"/>
 <vertex x="-1.905" y="40.005"/>
@@
 <wire x1="19.812" y1="68.072" x2="19.685" y2="68.005" width="0.4064" layer="1"/>
 <via x="19.812" y="69.596" extent="1-16" drill="0.3048"/>
-<polygon width="0.4064" layer="1">
+<polygon width="0.4064" layer="1" isolate="0.3048">
 <vertex x="-2.54" y="80.01"/>
 <vertex x="43.815" y="80.01"/>
@@
 <vertex x="-2.54" y="39.37"/>
 </polygon>
+<via x="27.94" y="52.07" extent="1-16" drill="0.3048"/>
+<via x="24.4475" y="52.07" extent="1-16" drill="0.3048"/>
+<via x="40.3225" y="63.1825" extent="1-16" drill="0.3048"/>
+<via x="40.64" y="57.15" extent="1-16" drill="0.3048"/>
 </signal>
 <signal name="VCC">
@@
 <wire x1="16.129" y1="70.485" x2="9.652" y2="64.008" width="0.4064" layer="1"/>
 <wire x1="38.608" y1="68.072" x2="36.195" y2="70.485" width="0.4064" layer="1"/>
-<wire x1="38.608" y1="55.372" x2="38.608" y2="68.072" width="0.4064" layer="1"/>
 <wire x1="38.1" y1="54.864" x2="38.608" y2="55.372" width="0.4064" layer="1"/>
 <wire x1="35.052" y1="54.864" x2="38.1" y2="54.864" width="0.4064" layer="1"/>
@@
 <wire x1="35.052" y1="54.864" x2="34.925" y2="54.9402" width="0.4064" layer="1"/>
 <wire x1="36.195" y1="70.485" x2="16.129" y2="70.485" width="0.4064" layer="1"/>
+<wire x1="38.608" y1="68.072" x2="38.608" y2="55.372" width="0.4064" layer="1"/>
 </signal>
 <signal name="N$4">
@@
 <wire x1="11.176" y1="66.548" x2="6.35" y2="66.548" width="0.4064" layer="1"/>
 <wire x1="15.748" y1="71.12" x2="11.176" y2="66.548" width="0.4064" layer="1"/>
-<wire x1="39.624" y1="53.848" x2="39.624" y2="68.326" width="0.4064" layer="1"/>
-<wire x1="38.1" y1="52.324" x2="39.624" y2="53.848" width="0.4064" layer="1"/>
-<wire x1="35.052" y1="52.324" x2="38.1" y2="52.324" width="0.4064" layer="1"/>
-<wire x1="35.052" y1="52.324" x2="34.925" y2="52.197" width="0.4064" layer="1"/>
-<wire x1="39.624" y1="68.326" x2="36.83" y2="71.12" width="0.4064" layer="1"/>
+<wire x1="39.37" y1="68.58" x2="36.83" y2="71.12" width="0.4064" layer="1"/>
 <wire x1="36.83" y1="71.12" x2="15.748" y2="71.12" width="0.4064" layer="1"/>
+<wire x1="39.37" y1="53.6575" x2="39.37" y2="68.58" width="0.4064" layer="1"/>
+<wire x1="34.925" y1="52.197" x2="37.9095" y2="52.197" width="0.4064" layer="1"/>
+<wire x1="37.9095" y1="52.197" x2="39.37" y2="53.6575" width="0.4064" layer="1"/>
 </signal>
 <signal name="N$5">
@@
 <wire x1="29.845" y1="71.755" x2="30.48" y2="72.39" width="0.4064" layer="1"/>
 <wire x1="37.465" y1="56.3118" x2="37.8968" y2="56.3118" width="0.4064" layer="16"/>
-<wire x1="37.8968" y1="56.3118" x2="41.91" y2="60.325" width="0.4064" layer="16"/>
 <wire x1="41.91" y1="60.325" x2="41.91" y2="64.77" width="0.4064" layer="16"/>
 <wire x1="5.715" y1="71.755" x2="2.54" y2="68.58" width="0.4064" layer="1"/>
 <wire x1="2.54" y1="68.58" x2="2.54" y2="63.7032" width="0.4064" layer="1"/>
 <wire x1="2.54" y1="63.7032" x2="3.81" y2="62.4332" width="0.4064" layer="1"/>
+<wire x1="37.8968" y1="56.3118" x2="41.91" y2="60.325" width="0.4064" layer="16"/>
 </signal>
 <signal name="N$14">
@@
 <contactref element="X1" pad="12"/>
 <contactref element="X2" pad="12"/>
-<wire x1="37.592" y1="58.928" x2="41.021" y2="62.357" width="0.4064" layer="16"/>
-<wire x1="37.592" y1="58.928" x2="37.465" y2="59.055" width="0.4064" layer="16"/>
-<via x="41.021" y="62.357" extent="1-16" drill="0.3048"/>
 <wire x1="36.83" y1="72.39" x2="33.02" y2="72.39" width="0.4064" layer="1"/>
 <wire x1="33.02" y1="72.39" x2="31.75" y2="73.66" width="0.4064" layer="1"/>
@@
 <wire x1="5.08" y1="72.39" x2="28.575" y2="72.39" width="0.4064" layer="1"/>
 <wire x1="28.575" y1="72.39" x2="29.845" y2="73.66" width="0.4064" layer="1"/>
-<wire x1="36.83" y1="72.39" x2="41.021" y2="68.199" width="0.4064" layer="1"/>
-<wire x1="41.021" y1="62.357" x2="41.021" y2="68.199" width="0.4064" layer="1"/>
+<wire x1="36.83" y1="72.39" x2="40.9575" y2="68.2625" width="0.4064" layer="1"/>
 <wire x1="5.08" y1="72.39" x2="1.27" y2="68.58" width="0.4064" layer="1"/>
 <wire x1="1.27" y1="68.58" x2="1.27" y2="62.23" width="0.4064" layer="1"/>
 <wire x1="1.27" y1="62.23" x2="3.81" y2="59.69" width="0.4064" layer="1"/>
+<wire x1="37.592" y1="58.928" x2="39.5605" y2="58.928" width="0.4064" layer="16"/>
+<wire x1="39.5605" y1="58.928" x2="41.275" y2="60.6425" width="0.4064" layer="16"/>
+<via x="40.9575" y="64.4525" extent="1-16" drill="0.3048"/>
+<wire x1="40.9575" y1="64.4525" x2="40.9575" y2="68.2625" width="0.4064" layer="1"/>
+<wire x1="37.592" y1="58.928" x2="37.465" y2="59.055" width="0.4064" layer="16"/>
+<wire x1="41.275" y1="60.6425" x2="41.275" y2="64.135" width="0.4064" layer="16"/>
+<wire x1="41.275" y1="64.135" x2="40.9575" y2="64.4525" width="0.4064" layer="16"/>
 </signal>
 <signal name="N$12">
@@
 <wire x1="12.065" y1="43.815" x2="10.16" y2="45.72" width="0.8128" layer="1"/>
 </signal>
-<signal name="N$17">
-<polygon width="0.8128" layer="16">
-<vertex x="-1.27" y="78.74"/>
-<vertex x="42.545" y="78.74"/>
-<vertex x="42.545" y="40.64"/>
-<vertex x="-1.27" y="40.64"/>
-</polygon>
-</signal>
-<signal name="N$18">
-<polygon width="0.4064" layer="1">
-<vertex x="-2.54" y="80.01"/>
-<vertex x="43.815" y="80.01"/>
-<vertex x="43.815" y="39.37"/>
-<vertex x="-2.54" y="39.37"/>
-</polygon>
-</signal>
 </signals>
