File: vga_ambilight_throughhole.brd (EAGLE design)
At the start: 46.4 x 40.6 mm, 16 parts, among them IC1 QUAD_OPAMPD

Commit message: commit
Parts:
- moved Q1 3.81 mm to (26.0, 53.3)
- moved Q2 3.81 mm to (22.2, 53.3)
- moved R1 3.81 mm to (26.0, 58.4)
- moved R2 3.81 mm to (22.2, 58.4)
Connections:
- net G_PWR: now also JP1.2, JP2.2, JP3.2, JP4.2; no longer JP1.3, JP2.3, JP3.3, JP4.3
- net R_PWR: now also JP1.3, JP2.3, JP3.3, JP4.3; no longer JP1.2, JP2.2, JP3.2, JP4.2
Routing:
- net N$8: track 10.0 -> 12.3 mm, vias 0 -> 2
- net N$7: track 5.96 -> 4.90 mm
- net R_PWR: track 12.0 -> 11.5 mm
- net G_PWR: track 11.5 -> 12.0 mm
Changed lines of the file:
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@@
 <attribute name="VALUE" x="-8.89" y="51.308" size="1.778" layer="27" ratio="10" rot="R90"/>
 </element>
-<element name="Q1" library="adafruit" package="SOT23" value="" x="22.225" y="53.34" smashed="yes" rot="R180">
+<element name="Q1" library="adafruit" package="SOT23" value="" x="26.035" y="53.34" smashed="yes" rot="R180">
+<attribute name="NAME" x="26.67" y="55.88" size="0.6096" layer="25" rot="R180"/>
+<attribute name="VALUE" x="27.94" y="56.515" size="1.27" layer="27" rot="R180"/>
+</element>
+<element name="Q2" library="adafruit" package="SOT23" value="" x="22.225" y="53.34" smashed="yes" rot="R180">
 <attribute name="NAME" x="22.86" y="55.88" size="0.6096" layer="25" rot="R180"/>
 <attribute name="VALUE" x="24.13" y="56.515" size="1.27" layer="27" rot="R180"/>
-</element>
-<element name="Q2" library="adafruit" package="SOT23" value="" x="26.035" y="53.34" smashed="yes" rot="R180">
-<attribute name="NAME" x="26.67" y="55.88" size="0.6096" layer="25" rot="R180"/>
-<attribute name="VALUE" x="27.94" y="56.515" size="1.27" layer="27" rot="R180"/>
 </element>
 <element name="Q3" library="adafruit" package="SOT23" value="" x="29.845" y="53.34" smashed="yes" rot="R180">
@@
 <attribute name="VALUE" x="31.75" y="56.515" size="1.27" layer="27" rot="R180"/>
 </element>
-<element name="R1" library="adafruit" package="M0805" value="" x="22.225" y="58.42" smashed="yes" rot="R270">
+<element name="R1" library="adafruit" package="M0805" value="" x="26.035" y="58.42" smashed="yes" rot="R270">
+<attribute name="NAME" x="27.305" y="59.69" size="1.27" layer="25" rot="R270"/>
+<attribute name="VALUE" x="23.495" y="59.69" size="1.27" layer="27" rot="R270"/>
+</element>
+<element name="R2" library="adafruit" package="M0805" value="" x="22.225" y="58.42" smashed="yes" rot="R270">
 <attribute name="NAME" x="23.495" y="59.69" size="1.27" layer="25" rot="R270"/>
 <attribute name="VALUE" x="19.685" y="59.69" size="1.27" layer="27" rot="R270"/>
-</element>
-<element name="R2" library="adafruit" package="M0805" value="" x="26.035" y="58.42" smashed="yes" rot="R270">
-<attribute name="NAME" x="27.305" y="59.69" size="1.27" layer="25" rot="R270"/>
-<attribute name="VALUE" x="23.495" y="59.69" size="1.27" layer="27" rot="R270"/>
 </element>
 <element name="R3" library="adafruit" package="M0805" value="" x="29.845" y="58.42" smashed="yes" rot="R270">
@@
 <wire x1="22.352" y1="62.992" x2="22.225" y2="62.805" width="0.4064" layer="1"/>
 <wire x1="23.368" y1="62.992" x2="23.495" y2="62.805" width="0.4064" layer="1"/>
-<wire x1="23.495" y1="62.805" x2="26.035" y2="60.265" width="0.4064" layer="1"/>
-<wire x1="26.035" y1="60.265" x2="26.035" y2="59.37" width="0.4064" layer="1"/>
+<wire x1="22.225" y1="59.37" x2="22.225" y2="62.805" width="0.4064" layer="1"/>
 </signal>
 <signal name="N$8">
@@
 <contactref element="IC1" pad="1"/>
 <contactref element="R1" pad="1"/>
-<wire x1="15.875" y1="62.805" x2="15.875" y2="61.595" width="0.4064" layer="1"/>
 <wire x1="15.875" y1="62.805" x2="17.145" y2="62.805" width="0.4064" layer="1"/>
-<wire x1="15.875" y1="61.595" x2="16.51" y2="60.96" width="0.4064" layer="1"/>
-<wire x1="16.51" y1="60.96" x2="18.415" y2="60.96" width="0.4064" layer="1"/>
-<wire x1="18.415" y1="60.96" x2="19.555" y2="59.82" width="0.4064" layer="1"/>
-<wire x1="19.555" y1="59.82" x2="22.225" y2="59.82" width="0.4064" layer="1"/>
-<wire x1="22.225" y1="59.82" x2="22.225" y2="59.37" width="0.4064" layer="1"/>
+<wire x1="17.145" y1="62.805" x2="17.145" y2="61.595" width="0.4064" layer="1"/>
+<wire x1="17.145" y1="61.595" x2="18.7325" y2="60.0075" width="0.4064" layer="1"/>
+<wire x1="18.7325" y1="60.0075" x2="19.05" y2="60.0075" width="0.4064" layer="1"/>
+<via x="19.05" y="60.0075" extent="1-16" drill="0.3048"/>
+<wire x1="19.05" y1="60.0075" x2="24.13" y2="60.0075" width="0.4064" layer="16"/>
+<via x="24.13" y="60.0075" extent="1-16" drill="0.3048"/>
+<wire x1="24.13" y1="60.0075" x2="25.3975" y2="60.0075" width="0.4064" layer="1"/>
+<wire x1="25.3975" y1="60.0075" x2="26.035" y2="59.37" width="0.4064" layer="1"/>
 </signal>
 <signal name="R">
@@
 <contactref element="Q1" pad="1"/>
 <contactref element="R1" pad="2"/>
-<wire x1="22.86" y1="56.388" x2="22.86" y2="54.864" width="0.4064" layer="1"/>
-<wire x1="22.352" y1="56.896" x2="22.86" y2="56.388" width="0.4064" layer="1"/>
-<wire x1="22.86" y1="54.864" x2="23.175" y2="54.44" width="0.4064" layer="1"/>
-<wire x1="22.352" y1="56.896" x2="22.225" y2="57.47" width="0.4064" layer="1"/>
+<wire x1="26.985" y1="54.44" x2="26.985" y2="56.52" width="0.4064" layer="1"/>
+<wire x1="26.985" y1="56.52" x2="26.035" y2="57.47" width="0.4064" layer="1"/>
 </signal>
 <signal name="N$13">
 <contactref element="Q2" pad="1"/>
 <contactref element="R2" pad="2"/>
-<wire x1="26.924" y1="56.388" x2="26.924" y2="54.864" width="0.4064" layer="1"/>
-<wire x1="26.416" y1="56.896" x2="26.924" y2="56.388" width="0.4064" layer="1"/>
-<wire x1="26.924" y1="54.864" x2="26.985" y2="54.44" width="0.4064" layer="1"/>
-<wire x1="26.416" y1="56.896" x2="26.035" y2="57.47" width="0.4064" layer="1"/>
+<wire x1="23.175" y1="54.44" x2="23.175" y2="56.52" width="0.4064" layer="1"/>
+<wire x1="23.175" y1="56.52" x2="22.225" y2="57.47" width="0.4064" layer="1"/>
 </signal>
 <signal name="N$16">
@@
 </signal>
 <signal name="R_PWR">
+<contactref element="Q1" pad="3"/>
+<contactref element="JP4" pad="3"/>
+<contactref element="JP3" pad="3"/>
+<contactref element="JP2" pad="3"/>
+<contactref element="JP2" pad="3"/>
+<contactref element="JP1" pad="3"/>
+<wire x1="27.305" y1="41.275" x2="27.305" y2="43.815" width="0.8128" layer="1"/>
+<wire x1="27.305" y1="43.815" x2="27.305" y2="46.355" width="0.8128" layer="1"/>
+<wire x1="27.305" y1="46.355" x2="27.305" y2="48.895" width="0.8128" layer="1"/>
+<wire x1="27.305" y1="48.895" x2="27.305" y2="50.97" width="0.8128" layer="1"/>
+<wire x1="27.305" y1="50.97" x2="26.035" y2="52.24" width="0.8128" layer="1"/>
+</signal>
+<signal name="G_PWR">
+<contactref element="Q2" pad="3"/>
 <contactref element="JP4" pad="2"/>
 <contactref element="JP3" pad="2"/>
@@
 <contactref element="JP2" pad="2"/>
 <contactref element="JP1" pad="2"/>
-<contactref element="Q1" pad="3"/>
-<wire x1="24.765" y1="48.895" x2="24.765" y2="46.355" width="0.8128" layer="1"/>
-<wire x1="24.765" y1="46.355" x2="24.765" y2="43.815" width="0.8128" layer="1"/>
-<wire x1="24.765" y1="43.815" x2="24.765" y2="41.275" width="0.8128" layer="1"/>
-<wire x1="22.225" y1="52.24" x2="22.225" y2="52.07" width="0.8128" layer="1"/>
-<wire x1="22.225" y1="52.07" x2="24.765" y2="49.53" width="0.8128" layer="1"/>
-<wire x1="24.765" y1="49.53" x2="24.765" y2="48.895" width="0.8128" layer="1"/>
-</signal>
-<signal name="G_PWR">
-<contactref element="JP4" pad="3"/>
-<contactref element="JP3" pad="3"/>
-<contactref element="JP2" pad="3"/>
-<contactref element="JP2" pad="3"/>
-<contactref element="JP1" pad="3"/>
-<contactref element="Q2" pad="3"/>
-<wire x1="27.305" y1="41.275" x2="27.305" y2="43.815" width="0.8128" layer="1"/>
-<wire x1="27.305" y1="43.815" x2="27.305" y2="46.355" width="0.8128" layer="1"/>
-<wire x1="27.305" y1="46.355" x2="27.305" y2="48.895" width="0.8128" layer="1"/>
-<wire x1="27.305" y1="48.895" x2="27.305" y2="50.165" width="0.8128" layer="1"/>
-<wire x1="27.305" y1="50.165" x2="26.035" y2="51.435" width="0.8128" layer="1"/>
-<wire x1="26.035" y1="51.435" x2="26.035" y2="52.24" width="0.8128" layer="1"/>
+<wire x1="24.765" y1="41.275" x2="24.765" y2="43.815" width="0.8128" layer="1"/>
+<wire x1="24.765" y1="43.815" x2="24.765" y2="46.355" width="0.8128" layer="1"/>
+<wire x1="24.765" y1="46.355" x2="24.765" y2="48.895" width="0.8128" layer="1"/>
+<wire x1="24.765" y1="48.895" x2="24.765" y2="49.7" width="0.8128" layer="1"/>
+<wire x1="24.765" y1="49.7" x2="22.225" y2="52.24" width="0.8128" layer="1"/>
 </signal>
 <signal name="B_PWR">
